Commit message: Add rigid RS485 wrist adapters to both hand models
Vendor the source GLB and runtime OBJ meshes, align the adapter screw holes, and preserve the attachment when rebuilding assets. Ignore temporary files and editor backups while retaining required model meshes.

File: assets/rh56e2_left.urdf (robot description, URDF)
Before this commit: robot rh56e2_left, 31 links, 30 joints
Links:
- link hand_base: geometry collision mesh filename=converted/left/base.obj scale=1 1 1; collision mesh filename=converted/left/wrist_rs485_adapter.obj scale=1 1 1

File: assets/rh56e2_right.urdf (robot description, URDF)
Before this commit: robot rh56e2_right, 31 links, 30 joints
Links:
- link hand_base: geometry collision mesh filename=converted/right/base.obj scale=1 1 1; collision mesh filename=converted/right/wrist_rs485_adapter.obj scale=1 1 1
